File: pcb/ponchos/motdrivhc05/motdrivhc05.kicad_pcb (KiCad board)
At the start: 2 copper layers, 25 parts, among them J1 MPower, J2 Screw_Terminal_1x04, J3 GW-040, J4 CONN_01X02, Q1 TIP31, Q2 TIP31, U1 L293

Commit message: Haciendo PCB...
Parts:
- moved C3 80.9 mm to (74.9, 36.8)
- moved C1 33.1 mm to (67.9, 38.1)
- moved C2 32.1 mm to (57.5, 39.1)
- moved D2 11.1 mm to (52.7, 78.7), turned to 0 degrees
- moved D6 11.0 mm to (62.9, 75.9), turned to 180 degrees
- moved D8 10.3 mm to (67.6, 84.5), turned to 0 degrees
- moved R2 10.2 mm to (93.3, 88.9), turned to 180 degrees
- moved D1 9.69 mm to (52.7, 84.5), turned to 0 degrees
- moved D7 8.82 mm to (67.6, 78.7), turned to 0 degrees
- moved D3 8.58 mm to (77.8, 75.9), turned to 180 degrees
- moved U1 6.68 mm to (63.8, 50.5)
- moved D4 6.11 mm to (77.8, 81.6), turned to 180 degrees
- moved D5 5.26 mm to (62.9, 81.6), turned to 180 degrees
- moved J2 2.73 mm to (65.7, 92.4)
Routing:
- net GND: track 0.00 -> 36.4 mm
- net /M4A: track 0.00 -> 29.8 mm
- net /M3A: track 0.00 -> 27.1 mm
- net /ME34: track 0.00 -> 26.6 mm
- net Net-(D1-Pad2): track 17.5 -> 42.7 mm
- net Net-(D2-Pad2): track 23.6 -> 48.5 mm
- net Net-(D3-Pad2): track 28.1 -> 47.1 mm
- net VCC: track 0.00 -> 14.9 mm
- net Net-(D4-Pad2): track 31.0 -> 43.7 mm
- net /BT_TXD: track 34.5 -> 33.0 mm
- net Net-(J3-Pad2): track 18.6 -> 17.5 mm
- net /BT_STATE: track 10.3 -> 9.68 mm
- added copper zone on B.Cu, net GND

Commit message: En desarrollo...
Parts:
- C1, C2: footprint Capacitors_ThroughHole:C_Radial_D7.5_L11.2_P2.5 -> Capacitors_ThroughHole:C_Radial_D6.3_L11.2_P2.5
- Q1, Q2: footprint TO_SOT_Packages_THT:TO-220_Neutral123_Horizontal_LargePads -> TO_SOT_Packages_THT:TO-220_Neutral123_Vertical_LargePads
- moved D9 76.7 mm to (76.8, 35.2), turned to 270 degrees
- moved R3 75.3 mm to (73.7, 35.2), turned to 270 degrees
- moved Q1 59.6 mm to (68.6, 39.4), turned to 270 degrees
- moved J1 49.9 mm to (57.1, 72.4), turned to 270 degrees
- moved Q2 33.9 mm to (55.9, 39.4), turned to 270 degrees
- moved R4 30.5 mm to (61.0, 35.2), turned to 270 degrees
- moved D10 29.8 mm to (64.1, 35.2), turned to 270 degrees
- moved C1 28.4 mm to (58.1, 64.8)
- moved J4 17.1 mm to (49.5, 52.1)
- moved C3 14.6 mm to (74.6, 51.4)
- moved C2 11.8 mm to (58.7, 50.8), turned to 180 degrees
- moved D2 4.13 mm to (52.7, 82.9)
- moved D3 4.13 mm to (77.8, 80.0)
- moved D6 4.13 mm to (62.9, 80.0)
- moved D7 4.13 mm to (67.6, 82.9)
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Connections:
- SH1 pad A4/2: /T2 -> /T1
- SH1 pad A5/2: /T1 -> /T2
Routing:
- net GND: track 36.4 -> 148.4 mm
- net VCC: track 14.9 -> 94.1 mm
- net Net-(D9-Pad1): track 0.00 -> 50.8 mm
- net +5V: track 0.00 -> 46.6 mm
- net /M2A: track 0.00 -> 43.9 mm, vias 0 -> 2
- net /T2: track 0.00 -> 42.3 mm
- net Net-(D10-Pad1): track 0.00 -> 29.9 mm
- net /M4A: track 29.8 -> 0.00 mm
- net /T1: track 0.00 -> 29.5 mm
- net /M3A: track 27.1 -> 0.00 mm
- net /ME34: track 26.6 -> 0.00 mm
- net Net-(Q1-Pad1): track 0.00 -> 6.00 mm
- net Net-(Q2-Pad1): track 0.00 -> 5.74 mm
- net Net-(D4-Pad2): track 43.7 -> 48.3 mm
- net Net-(D3-Pad2): track 47.1 -> 49.1 mm
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
Commit message: En proceso...
Parts:
- removed D10: 1N5819, Diodes_ThroughHole:Diode_DO-41_SOD81_Horizontal_RM10
- removed Q2: TIP31, TO_SOT_Packages_THT:TO-220_Neutral123_Vertical_LargePads
- removed R4: 1K, Resistors_ThroughHole:Resistor_Horizontal_RM10mm
- moved C2 18.8 mm to (75.9, 43.2), turned to 90 degrees
- moved D9 17.1 mm to (60.6, 40.6), turned to 0 degrees
- moved R3 15.8 mm to (60.6, 44.1), turned to 0 degrees
- moved Q1 14.3 mm to (55.9, 46.0)
- moved J4 3.84 mm to (51.1, 55.6), turned to 180 degrees
- moved R1 1.14 mm to (94.3, 92.7)
- moved R2 0.95 mm to (94.3, 88.9)
Connections:
- J4 pad 1: Net-(D9-Pad1) -> Net-(J4-Pad1)
- J4 pad 2: Net-(D10-Pad1) -> Net-(D9-Pad1)
Routing:
- net GND: track 148.4 -> 214.0 mm
- net /M1A: track 0.00 -> 52.3 mm, vias 0 -> 2
- net /ME12: track 0.00 -> 50.1 mm, vias 0 -> 2
- net /T2: track 42.3 -> 0.00 mm
- net /M3A: track 0.00 -> 31.0 mm, vias 0 -> 2
- net Net-(D10-Pad1): track 29.9 -> 0.00 mm
- net Net-(D9-Pad1): track 50.8 -> 22.1 mm
- net /ME34: track 0.00 -> 27.7 mm, vias 0 -> 2
- net +5V: track 46.6 -> 71.2 mm
- net /M2A: track 43.9 -> 55.0 mm
- net Net-(Q2-Pad1): track 5.74 -> 0.00 mm
- net /BT_TXD: track 33.1 -> 30.1 mm
- net /T1: track 29.5 -> 31.0 mm, vias 0 -> 2
- net Net-(Q1-Pad1): track 6.00 -> 5.03 mm
- net /BT_RXD: track 4.45 -> 3.76 mm
Other:
- board outline added: 53.3 x 64.1 mm

Commit message: En processo...
Parts:
- removed J2: Screw_Terminal_1x04, Connect:bornier4
- J1: value MPower -> Screw_Terminal_1x06; footprint Connect:bornier2 -> Terminal_Blocks:TerminalBlock_Pheonix_MKDS1.5-6pol
- moved J1 19.3 mm to (54.0, 91.4), turned to 0 degrees
- moved R2 6.26 mm to (88.9, 85.7), turned to 270 degrees
- moved C1 5.85 mm to (59.4, 70.5), turned to 180 degrees
- moved D2 4.14 mm to (53.0, 78.7)
- moved D3 4.14 mm to (78.1, 75.9)
- moved D6 4.14 mm to (63.2, 75.9)
- moved D7 4.14 mm to (67.9, 78.7)
- moved D4 4.14 mm to (78.1, 81.6)
- moved D1 4.14 mm to (53.0, 84.5)
- moved D5 4.14 mm to (63.2, 81.6)
- moved D8 4.14 mm to (67.9, 84.5)
- moved R1 3.55 mm to (92.7, 95.9), turned to 90 degrees
- moved J3 1.62 mm to (94.3, 82.2)
Connections:
- J1 pad 1: VCC -> GND
- J1 pad 2: GND -> VCC
Routing:
- net GND: track 214.0 -> 257.6 mm
- net /M4A: track 0.00 -> 30.8 mm, vias 0 -> 4
- net Net-(D3-Pad2): track 49.1 -> 38.0 mm
- net Net-(J3-Pad2): track 17.2 -> 7.27 mm
- net Net-(D2-Pad2): track 49.8 -> 40.6 mm
- net VCC: track 94.1 -> 86.3 mm
- net /BT_TXD: track 30.1 -> 25.3 mm
- net /ME12: track 50.1 -> 53.9 mm
- net /M1A: track 52.3 -> 55.7 mm
- net /BT_RXD: track 3.76 -> 7.03 mm
- net /BT_STATE: track 9.68 -> 10.8 mm
- net /M2A: track 55.0 -> 55.9 mm

Commit message: Primer versión de PCB terminada.
Parts:
- moved C1 16.9 mm to (44.1, 63.2)
- moved J4 16.2 mm to (35.6, 51.1)
- moved C2 15.8 mm to (61.0, 38.1)
- moved D3 15.6 mm to (63.2, 71.4)
- moved D4 15.6 mm to (63.2, 77.2)
- moved J3 15.6 mm to (79.4, 77.8)
- moved R1 15.6 mm to (77.8, 91.4)
- moved D1 15.6 mm to (38.1, 80.0)
- moved D2 15.6 mm to (38.1, 74.3)
- moved D5 15.6 mm to (48.3, 77.2)
- moved D6 15.6 mm to (48.3, 71.4)
- moved Q1 15.6 mm to (41.0, 41.6)
- moved R2 15.6 mm to (74.0, 81.3)
- moved SH1 15.6 mm to (58.7, 62.2)
- moved U1 15.6 mm to (48.9, 46.0)
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Routing:
- net +5V: track 71.4 -> 166.5 mm, vias 0 -> 2
- net VCC: track 86.3 -> 100.5 mm
- net GND: track 257.6 -> 270.8 mm
- net Net-(D1-Pad2): track 44.6 -> 46.9 mm
- net /M3A: track 31.0 -> 32.8 mm
- net Net-(D4-Pad2): track 48.7 -> 50.5 mm
- net /ME34: track 27.7 -> 29.0 mm
- net /ME12: track 53.9 -> 54.9 mm
- net /M1A: track 55.7 -> 54.7 mm
- net /BT_RXD: track 7.03 -> 6.13 mm
- net Net-(D3-Pad2): track 38.0 -> 38.7 mm
Other:
- board size 53.3 x 64.1 mm -> 53.3 x 61.6 mm
