File: pcb/ponchos/acelerometro_leds_rele/Shield superior.kicad_pcb (KiCad board)
At the start: 2 copper layers, 54.4 x 56.7 mm, 13 parts, among them J1 CONN_01X08, J2 CONN_01X06, J3 CONN_01X10, J4 CONN_01X08, J5 CONN_01X03, J6 Screw_Terminal_1x03, J7 CONN_01X08, K1 AZ850-x, Q1 BC548, U1 7805

Commit message: Modificaciones al shield superior, mejora en conexión del acelerómetro y ajueste de distancias en el ponout del arduino.
Parts:
- D1: footprint Diodes_THT:D_5W_P12.70mm_Horizontal -> Diodes_THT:D_5W_P10.16mm_Horizontal
- R1, R2: footprint Resistors_THT:R_Axial_DIN0309_L9.0mm_D3.2mm_P12.70mm_Horizontal -> Resistors_THT:R_Axial_DIN0207_L6.3mm_D2.5mm_P7.62mm_Horizontal
- moved J7 24.0 mm to (29.7, 74.5), turned to 90 degrees
- moved R2 16.9 mm to (63.7, 55.7)
- moved R1 15.5 mm to (56.0, 51.0)
- moved J5 4.49 mm to (57.3, 62.1)
- moved J4 0.42 mm to (72.4, 57.1)
- turned Q1 to 0 degrees
Routing:
- net /Data: track 16.7 -> 7.08 mm
- net /SDA: track 22.1 -> 13.2 mm
- net Net-(Q1-Pad2): track 19.3 -> 11.7 mm
- net +5V: track 77.2 -> 84.4 mm
- net Net-(J4-Pad2): track 16.7 -> 10.4 mm
- net /INT: track 44.0 -> 49.2 mm
- net Net-(J4-Pad1): track 13.7 -> 11.4 mm
- net /SCL: track 23.3 -> 25.5 mm, vias 2 -> 0

Commit message: Modifico para agrandar margen a 0,6 huellas y símbolos dentro del proyecto.
Parts:
- D1: footprint Diodes_THT:D_5W_P10.16mm_Horizontal -> huellas:D_5W_P10.16mm_Horizontal
- J1, J4, J7: footprint Connectors_JST:JST_EH_B08B-EH-A_08x2.50mm_Straight -> huellas:JST_EH_B08B-EH-A_08x2.50mm_Straight
- J2: footprint Connectors_JST:JST_EH_B06B-EH-A_06x2.50mm_Straight -> huellas:JST_EH_B06B-EH-A_06x2.50mm_Straight
- J3: footprint Connectors_JST:JST_EH_B10B-EH-A_10x2.50mm_Straight -> huellas:JST_EH_B10B-EH-A_10x2.50mm_Straight
- J5: footprint Connectors_JST:JST_EH_B03B-EH-A_03x2.50mm_Straight -> huellas:JST_EH_B03B-EH-A_03x2.50mm_Straight
- J6: footprint Connectors_Terminal_Blocks:TerminalBlock_Pheonix_MKDS1.5-3pol -> huellas:TerminalBlock_Pheonix_MKDS1.5-3pol
- K1: footprint Relays_THT:Relay_THT_5V -> huellas:Relay_THT_5V
- Q1: footprint TO_SOT_Packages_THT:TO-92_Molded_Narrow -> TO_SOT_Packages_THT:TO-92_Inline_Wide
- R1, R2: footprint Resistors_THT:R_Axial_DIN0207_L6.3mm_D2.5mm_P7.62mm_Horizontal -> huellas:R_Axial_DIN0207_L6.3mm_D2.5mm_P7.62mm_Horizontal
- U1: footprint TO_SOT_Packages_THT:TO-220_Vertical -> huellas:TO-220_Vertical
- moved U1 6.72 mm to (24.8, 31.0), turned to 90 degrees
- moved Q1 1.51 mm to (43.5, 50.0)
Connections:
- U1 pad 1: /Vin -> +5V
- U1 pad 3: +5V -> /Vin
Routing:
- net Net-(D1-Pad2): track 17.5 -> 19.7 mm
- net +5V: track 84.4 -> 82.6 mm
- net Net-(Q1-Pad2): track 11.7 -> 13.2 mm
- net /Vin: track 34.7 -> 35.7 mm
Other:
- board size 54.4 x 56.7 mm -> 55 x 57 mm
- net class Default: clearance 0.2 -> 0.6
- net class Via2 removed
- rule trace_clearance: 0.2 -> 0.6
- board text added: "5V"
- board text added: "D"
- board text added: "GND"
- board text added: "UNLaM LACIE 2018"
